File: wiring/wiring.kicad_sch (KiCad schematic)
At the start: 0 parts

Commit message: AVR and RPI wired together
Parts:
- added U1: (no value), symbol CustomSymbols:AVR64DU32_Curiosity_Nano
- added U2: (no value), symbol CustomSymbols:RPI4B_Extended
Connections:
- new net: U1. (NC), U2. (USB03)
- new net: U2.1 (3V3), U2.17 (3V3)
- new net: U2.14 (GND), U2.20 (GND), U2.25 (GND), U2.30 (GND), U2.34 (GND), U2.39 (GND), U2.6 (GND), U2.9 (GND)
- new net: U2.2 (5V), U2.4 (5V)

Commit message: completed kicad diagram
Parts:
- added BTN_LCLICK, BTN_LCLICKHOLD, BTN_QUIT, BTN_VIRTKBD: SW_Push, symbol Switch:SW_Push
- added KNOB_X, KNOB_Y: RotaryEncoder, symbol Device:RotaryEncoder
- added LED_LCLICK, LED_PWR, LED_SHAKE: LED, symbol Device:LED
- added R1, R2, R3: 160, symbol Device:R
- added U3: (no value), symbol CustomSymbols:Adafruit_HUSB238_USB_Type_C_Power_Delivery_Breakout
- added U4: LSM6DSOTR, LGA-14L_2P5X3X0P86_STM, symbol LSM6DSO:LSM6DSOTR
Connections:
- net GND: now reaches U1. (NC)
- net GND: now also BTN_LCLICK.1, BTN_LCLICKHOLD.1, BTN_QUIT.1, BTN_VIRTKBD.1, KNOB_X.C, KNOB_Y.C, R1.1, R2.1, R3.1, U4.6 (GND)
- net at U2. (USB03): no longer U1. (NC)
- net at U2.14 (GND), U2.20 (GND), U2.25 (GND)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: now also U3. (18V+)
- net at U2.2 (5V), U2.4 (5V): now also U3. (18V+)
- new net: LED_SHAKE.1 (K), R1.2
- new net: LED_SHAKE.2 (A), U1. (NC)
- new net: U1. (NC), U4.13 (SCL)
- new net: U1. (NC), U4.14 (SDA)
- new net: U1. (NC), U4.8 (VDD)
- new net: LED_PWR.1 (K), R3.2
- new net: LED_LCLICK.1 (K), R2.2
- new net: LED_LCLICK.2 (A), U1. (NC)
- new net: U1. (NC), U2. (USB03)
- new net: BTN_VIRTKBD.2, U1. (NC)
- new net: BTN_LCLICK.2, U1. (NC)
- new net: LED_PWR.2 (A), U1. (NC)
- new net: KNOB_X.A, U1. (NC)
- new net: KNOB_X.B, U1. (NC)
- new net: BTN_LCLICKHOLD.2, U1. (NC)
- new net: KNOB_Y.A, U1. (NC)
- new net: KNOB_Y.B, U1. (NC)
- new net: BTN_QUIT.2, U1. (NC)
- new net USB_PD_PWR: U3. (18V+)
Other:
- note added: "USE ONLY THIS GND"
- moved on the sheet: U1, U2

Commit message: missing DSI Display
Parts:
- added U5: (no value), symbol CustomSymbols:DSI_Display
Connections:
- net at U2. (USB03): now also U5.; no longer U1. (NC)
- new net: U1. (NC), U2. (USB03)
Changed lines of the file:
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@@
+	(wire
+		(pts
+			(xy 34.29 105.41) (xy 44.45 105.41)
+		)
+		(stroke
+			(width 0)
+			(type default)
+		)
+	)
 	(wire
 		(pts
@@
 		(pin "5"
 		)
+		(pin ""
+		)
 		(instances
 			(project "wiring"
@@
 					(unit 1)
 				)
+			)
+		)
+	)
+	(symbol
+		(lib_id "CustomSymbols:DSI_Display")
+		(at 34.29 99.06 0)
+		(unit 1)
+		(body_style 1)
+		(exclude_from_sim no)
+		(in_bom yes)
+		(on_board yes)
+		(in_pos_files yes)
+		(dnp no)
+		(fields_autoplaced yes)
+		(property "Reference" "U5"
+			(at 34.29 97.79 0)
+			(show_name no)
+			(do_not_autoplace no)
+			(effects
+				(font
+					(size 1.27 1.27)
+				)
+			)
+		)
+		(property "Value" ""
+			(at 34.29 99.06 0)
+			(show_name no)
+			(do_not_autoplace no)
+			(effects
+				(font
+					(size 1.27 1.27)
+				)
+			)
+		)
+		(property "Footprint" ""
+			(at 34.29 99.06 0)
+			(hide yes)
+			(show_name no)
+			(do_not_autoplace no)
+			(effects
+				(font
+					(size 1.27 1.27)
+				)
+			)
+		)
+		(property "Datasheet" ""
+			(at 34.29 99.06 0)
+			(hide yes)
+			(show_name no)
+			(do_not_autoplace no)
+			(effects
+				(font
+					(size 1.27 1.27)
+				)
+			)
+		)
+		(property "Description" ""
+			(at 34.29 99.06 0)
+			(hide yes)
+			(show_name no)
+			(do_not_autoplace no)
+			(effects
+				(font
+					(size 1.27 1.27)
+				)
+			)
+		)
+		(pin ""
+		)
+		(instances
+			(project "wiring"
+				(path "/2e6e7072-ae9c-40cf-83f0-1223d4dd0915"
+					(reference "U5")
+					(unit 1)
+				)
